File: PowerampC300/PowerampC300.kicad_pcb (KiCad board)
At the start: 2 copper layers, 240 x 63 mm, 95 parts, among them J1 Conn_01x02, J2 Conn_01x02, J3 Conn_01x02, J4 Conn_01x01, J5 Conn_01x01, J6 Conn_01x01, J7 Conn_01x01, J8 Conn_01x02, J9 Conn_Coaxial, Q1 BC546, Q10 MJE350, Q11 MJE340, Q12 MJE340, Q13 BC546, Q14 BC556, Q15 MJE340, Q16 MJE350, Q17 MJL3281A, Q18 MJL1302A, Q19 MJL3281A, Q2 BC546, Q20 MJL1302A, Q21 MJL3281A, Q22 MJL1302A, Q23 MJL3281A, Q24 MJL1302A, Q3 BC556, Q4 BC556, Q5 BC546, Q6 BC546, Q7 BC546, Q8 MPSA92, Q9 BC556

Commit message: Added power condition board
Parts:
- moved C4 15.0 mm to (90.0, 102.0), turned to 90 degrees
- moved C7 14.6 mm to (55.5, 99.2)
- moved C8 13.0 mm to (38.8, 99.2)
- moved R13 4.00 mm to (90.0, 89.0)
- moved Q12 2.00 mm to (161.0, 80.0)
- moved R18 1.12 mm to (124.0, 73.0)
- moved R25 1.12 mm to (129.0, 69.0)
- moved R26 1.00 mm to (134.0, 73.0)
Routing:
- net Net-(C7-Pad1): track 9.37 -> 15.5 mm
- net Net-(C7-Pad2): track 10.5 -> 6.75 mm
- net +48V: track 261.8 -> 265.5 mm
- net Net-(C4-Pad2): track 29.6 -> 27.0 mm
- net Net-(C5-Pad2): track 35.5 -> 37.1 mm
- net Net-(C10-Pad1): track 61.2 -> 60.0 mm
- net Net-(Q9-Pad3): track 7.34 -> 8.34 mm
- net OUTPUT: track 390.1 -> 389.1 mm
- net Net-(Q13-Pad2): track 13.4 -> 12.6 mm
- net Net-(Q12-Pad1): track 14.3 -> 14.8 mm

Commit message: Added XLRtoBal
Parts:
- removed R25: 3k3, Resistors_THT:R_Axial_DIN0411_L9.9mm_D3.6mm_P15.24mm_Horizontal
- moved R18 7.43 mm to (117.2, 76.0), turned to 90 degrees
- moved R17 7.26 mm to (109.1, 76.2)
- moved R19 4.81 mm to (113.2, 76.2)
- moved C10 3.42 mm to (152.6, 85.6)
- moved Q9 3.38 mm to (114.3, 81.8)
- moved R20 3.34 mm to (117.0, 85.0)
- moved C2 3.27 mm to (130.9, 95.2)
- moved Q11 3.00 mm to (153.0, 73.0)
- moved R1 2.88 mm to (123.3, 98.4)
- moved R6 2.63 mm to (134.6, 101.6)
- moved R7 2.17 mm to (134.6, 104.1)
- moved C9 1.95 mm to (116.6, 93.3)
- moved Q10 1.94 mm to (126.5, 86.9)
- moved R23 0.26 mm to (152.3, 89.0)
Routing:
- net +48V: track 265.5 -> 248.2 mm
- net Net-(Q10-Pad3): track 27.5 -> 37.1 mm
- net Net-(Q9-Pad2): track 8.12 -> 12.9 mm
- net Net-(C10-Pad1): track 60.0 -> 64.5 mm
- net Net-(Q9-Pad3): track 8.34 -> 4.51 mm
- net Net-(Q10-Pad1): track 6.90 -> 10.7 mm
- net Net-(C9-Pad1): track 29.8 -> 27.3 mm
- net Net-(R10-Pad3): track 12.7 -> 15.1 mm
- net Net-(C1-Pad1): track 19.1 -> 21.5 mm
- net Net-(Q11-Pad3): track 13.7 -> 15.2 mm
- net Net-(Q1-Pad3): track 11.3 -> 12.1 mm
- net Net-(R10-Pad1): track 12.5 -> 13.4 mm
- net Net-(C10-Pad2): track 86.7 -> 86.1 mm
- net Net-(Q2-Pad3): track 19.8 -> 20.3 mm
- added copper zone on B.Cu, net +48V
- added copper zone on B.Cu, net -48V
- added copper zone on F.Cu, net OUTPUT

Commit message: Added credit where credit is due
Parts:
- added C16: 100 uF, Capacitors_THT:CP_Radial_D14.0mm_P7.50mm, F.Cu at (35.8, 75.0)
- added C17: 100 uF, Capacitors_THT:CP_Radial_D14.0mm_P7.50mm, F.Cu at (39.5, 90.5)
- added C18: 100 uF, Capacitors_THT:CP_Radial_D14.0mm_P7.50mm, F.Cu at (220.0, 89.5)
- added C19: 100 uF, Capacitors_THT:CP_Radial_D14.0mm_P7.50mm, F.Cu at (197.2, 89.5)
- added R25: 3k3, Resistors_THT:R_Axial_DIN0411_L9.9mm_D3.6mm_P15.24mm_Horizontal, F.Cu at (132.5, 73.5)
- moved C8 22.6 mm to (54.2, 82.8), turned to 270 degrees
- moved R26 7.00 mm to (128.2, 69.0)
- moved R16 6.02 mm to (190.5, 91.5), turned to 270 degrees
- moved J1 5.81 mm to (247.8, 74.5)
- moved J2 5.71 mm to (231.0, 74.8)
- moved R18 4.45 mm to (112.8, 76.0)
- moved R19 4.23 mm to (109.0, 76.0)
- moved R17 4.13 mm to (105.0, 76.0)
- moved R3 3.54 mm to (101.0, 76.0)
- moved R4 3.04 mm to (96.0, 76.0)
- moved R15 2.46 mm to (66.8, 93.5)
- moved R41 2.00 mm to (58.0, 77.5)
- moved R13 1.75 mm to (90.0, 87.2)
- moved C7 1.35 mm to (54.2, 98.8), turned to 90 degrees
Routing:
- net +48V: track 248.2 -> 302.0 mm
- net -48V: track 265.5 -> 299.8 mm
- net Net-(C5-Pad2): track 37.1 -> 41.7 mm
- net Net-(C6-Pad1): track 40.9 -> 44.4 mm
- net Net-(Q13-Pad2): track 12.6 -> 15.8 mm
- net Net-(Q3-Pad3): track 3.46 -> 5.58 mm
- net Net-(C4-Pad2): track 27.0 -> 28.8 mm
- net OUTPUT: track 389.1 -> 390.5 mm
- net Net-(Q9-Pad2): track 12.9 -> 14.1 mm
- net Net-(C7-Pad1): track 15.5 -> 14.7 mm
- net Net-(C7-Pad2): track 6.75 -> 6.00 mm
- net Net-(C11-Pad1): track 5.05 -> 5.75 mm
- net Net-(Q10-Pad3): track 37.1 -> 36.6 mm
- net Net-(Q4-Pad3): track 4.08 -> 4.58 mm
Other:
- board text added: "C300 AMPLIFIER PCB BY DANIEL MARKS C300 DESIGNED BY MICHAEL CHUA (AMPSLAB) CC-BY-SA 4.0"
- board text removed: "C300 AMPLIFIER PCB BY DANIEL MARKS CC-BY-SA 4.0"

Commit message: Added soft start circuit
Parts:
- added C20: 0.1 uF, Capacitors_THT:C_Disc_D5.0mm_W2.5mm_P5.00mm, F.Cu at (263.0, 92.2)
- added C21: 0.1 uF, Capacitors_THT:C_Disc_D5.0mm_W2.5mm_P5.00mm, F.Cu at (29.0, 92.5)
Connections:
- J2 pad 2: (no net) -> GND
- J4 pad 1: (no net) -> Net-(C20-Pad2)
- J6 pad 1: (no net) -> Net-(C21-Pad2)
Routing:
- net Net-(C20-Pad2): track 0.00 -> 5.75 mm
- net Net-(C21-Pad2): track 0.00 -> 5.50 mm
- net Net-(Q16-Pad1): track 161.2 -> 159.4 mm
Changed lines of the file:
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@@
 (kicad_pcb (version 4) (host pcbnew 4.0.7)
   (general
-    (links 192)
+    (links 197)
     (no_connects 0)
-    (area 24.252381 42.025 267.74762 107.905)
+    (area 25.924999 42.924999 266.075001 106.075001)
     (thickness 1.6)
     (drawings 18)
-    (tracks 531)
+    (tracks 533)
     (zones 0)
-    (modules 99)
-    (nets 51)
+    (modules 101)
+    (nets 53)
   )
   (page A4)
@@
   )
   (setup
-    (last_trace_width 0.5)
+    (last_trace_width 0.25)
     (user_trace_width 0.5)
     (user_trace_width 1)
@@
     (mod_text_size 1 1)
     (mod_text_width 0.15)
-    (pad_size 4.3 4.5)
-    (pad_drill 1.5)
+    (pad_size 5.5 5.5)
+    (pad_drill 3.048)
     (pad_to_mask_clearance 0.2)
     (aux_axis_origin 0 0)
@@
   (net 49 "Net-(R10-Pad2)")
   (net 50 "Net-(R22-Pad1)")
+  (net 51 "Net-(C20-Pad2)")
+  (net 52 "Net-(C21-Pad2)")
   (net_class Default "This is the default net class."
     (clearance 0.2)
@@
     (add_net "Net-(C11-Pad1)")
     (add_net "Net-(C2-Pad2)")
+    (add_net "Net-(C20-Pad2)")
+    (add_net "Net-(C21-Pad2)")
     (add_net "Net-(C3-Pad1)")
     (add_net "Net-(C3-Pad2)")
@@
     (pad 1 thru_hole rect (at 0 0) (size 3 3) (drill 1.52) (layers *.Cu *.Mask)
       (net 8 -48V))
-    (pad 2 thru_hole circle (at 5.08 0) (size 3 3) (drill 1.52) (layers *.Cu *.Mask))
+    (pad 2 thru_hole circle (at 5.08 0) (size 3 3) (drill 1.52) (layers *.Cu *.Mask)
+      (net 3 GND))
     (model ${KISYS3DMOD}/Terminal_Blocks.3dshapes/TerminalBlock_bornier-2_P5.08mm.wrl
       (at (xyz 0.1 0 0))
@@
     (fp_circle (center 0 0) (end 2.6 0) (layer F.CrtYd) (width 0.05))
     (fp_circle (center 0 0) (end 0 -2.286) (layer F.SilkS) (width 0.12))
-    (pad 1 thru_hole circle (at 0 0) (size 4.064 4.064) (drill 3.048) (layers *.Cu *.Mask))
+    (pad 1 thru_hole circle (at 0 0) (size 5.5 5.5) (drill 3.048) (layers *.Cu *.Mask)
+      (net 51 "Net-(C20-Pad2)"))
   )
   (module Connectors:1pin (layer F.Cu)
@@
     (fp_circle (center 0 0) (end 2.6 0) (layer F.CrtYd) (width 0.05))
     (fp_circle (center 0 0) (end 0 -2.286) (layer F.SilkS) (width 0.12))
-    (pad 1 thru_hole circle (at 0 0) (size 4.064 4.064) (drill 3.048) (layers *.Cu *.Mask))
+    (pad 1 thru_hole circle (at 0 0) (size 5.5 5.5) (drill 3.048) (layers *.Cu *.Mask)
+      (net 52 "Net-(C21-Pad2)"))
   )
   (module Connectors:1pin (layer F.Cu)
@@
     )
   )
+  (module Capacitors_THT:C_Disc_D5.0mm_W2.5mm_P5.00mm (layer F.Cu)
+    (at 263 92.25 270)
+    (descr "C, Disc series, Radial, pin pitch=5.00mm, , diameter*width=5*2.5mm^2, Capacitor, http://cdn-reichelt.de/documents/datenblatt/B300/DS_KERKO_TC.pdf")
+    (tags "C Disc series Radial pin pitch 5.00mm  diameter 5mm width 2.5mm Capacitor")
+    (fp_text reference C20 (at 2.5 0 270) (layer F.SilkS)
+      (effects (font (size 1 1) (thickness 0.15)))
+    )
+    (fp_text value "0.1 uF" (at 2.5 2.56 270) (layer F.Fab)
+      (effects (font (size 1 1) (thickness 0.15)))
+    )
+    (fp_line (start 0 -1.25) (end 0 1.25) (layer F.Fab) (width 0.1))
+    (fp_line (start 0 1.25) (end 5 1.25) (layer F.Fab) (width 0.1))
+    (fp_line (start 5 1.25) (end 5 -1.25) (layer F.Fab) (width 0.1))
+    (fp_line (start 5 -1.25) (end 0 -1.25) (layer F.Fab) (width 0.1))
+    (fp_line (start -0.06 -1.31) (end 5.06 -1.31) (layer F.SilkS) (width 0.12))
+    (fp_line (start -0.06 1.31) (end 5.06 1.31) (layer F.SilkS) (width 0.12))
+    (fp_line (start -0.06 -1.31) (end -0.06 -0.996) (layer F.SilkS) (width 0.12))
+    (fp_line (start -0.06 0.996) (end -0.06 1.31) (layer F.SilkS) (width 0.12))
+    (fp_line (start 5.06 -1.31) (end 5.06 -0.996) (layer F.SilkS) (width 0.12))
+    (fp_line (start 5.06 0.996) (end 5.06 1.31) (layer F.SilkS) (width 0.12))
+    (fp_line (start -1.05 -1.6) (end -1.05 1.6) (layer F.CrtYd) (width 0.05))
+    (fp_line (start -1.05 1.6) (end 6.05 1.6) (layer F.CrtYd) (width 0.05))
+    (fp_line (start 6.05 1.6) (end 6.05 -1.6) (layer F.CrtYd) (width 0.05))
+    (fp_line (start 6.05 -1.6) (end -1.05 -1.6) (layer F.CrtYd) (width 0.05))
+    (fp_text user %R (at 2.5 0 270) (layer F.Fab)
+      (effects (font (size 1 1) (thickness 0.15)))
+    )
+    (pad 1 thru_hole circle (at 0 0 270) (size 1.6 1.6) (drill 0.8) (layers *.Cu *.Mask)
+      (net 3 GND))
+    (pad 2 thru_hole circle (at 5 0 270) (size 1.6 1.6) (drill 0.8) (layers *.Cu *.Mask)
+      (net 51 "Net-(C20-Pad2)"))
+    (model ${KISYS3DMOD}/Capacitors_THT.3dshapes/C_Disc_D5.0mm_W2.5mm_P5.00mm.wrl
+      (at (xyz 0 0 0))
+      (scale (xyz 1 1 1))
+      (rotate (xyz 0 0 0))
+    )
+  )
+  (module Capacitors_THT:C_Disc_D5.0mm_W2.5mm_P5.00mm (layer F.Cu)
+    (at 29 92.5 270)
+    (descr "C, Disc series, Radial, pin pitch=5.00mm, , diameter*width=5*2.5mm^2, Capacitor, http://cdn-reichelt.de/documents/datenblatt/B300/DS_KERKO_TC.pdf")
+    (tags "C Disc series Radial pin pitch 5.00mm  diameter 5mm width 2.5mm Capacitor")
+    (fp_text reference C21 (at 2.5 0 270) (layer F.SilkS)
+      (effects (font (size 1 1) (thickness 0.15)))
+    )
+    (fp_text value "0.1 uF" (at 2.5 2.56 270) (layer F.Fab)
+      (effects (font (size 1 1) (thickness 0.15)))
+    )
+    (fp_line (start 0 -1.25) (end 0 1.25) (layer F.Fab) (width 0.1))
+    (fp_line (start 0 1.25) (end 5 1.25) (layer F.Fab) (width 0.1))
+    (fp_line (start 5 1.25) (end 5 -1.25) (layer F.Fab) (width 0.1))
+    (fp_line (start 5 -1.25) (end 0 -1.25) (layer F.Fab) (width 0.1))
+    (fp_line (start -0.06 -1.31) (end 5.06 -1.31) (layer F.SilkS) (width 0.12))
+    (fp_line (start -0.06 1.31) (end 5.06 1.31) (layer F.SilkS) (width 0.12))
+    (fp_line (start -0.06 -1.31) (end -0.06 -0.996) (layer F.SilkS) (width 0.12))
+    (fp_line (start -0.06 0.996) (end -0.06 1.31) (layer F.SilkS) (width 0.12))
+    (fp_line (start 5.06 -1.31) (end 5.06 -0.996) (layer F.SilkS) (width 0.12))
+    (fp_line (start 5.06 0.996) (end 5.06 1.31) (layer F.SilkS) (width 0.12))
+    (fp_line (start -1.05 -1.6) (end -1.05 1.6) (layer F.CrtYd) (width 0.05))
+    (fp_line (start -1.05 1.6) (end 6.05 1.6) (layer F.CrtYd) (width 0.05))
+    (fp_line (start 6.05 1.6) (end 6.05 -1.6) (layer F.CrtYd) (width 0.05))
+    (fp_line (start 6.05 -1.6) (end -1.05 -1.6) (layer F.CrtYd) (width 0.05))
+    (fp_text user %R (at 2.5 0 270) (layer F.Fab)
+      (effects (font (size 1 1) (thickness 0.15)))
+    )
+    (pad 1 thru_hole circle (at 0 0 270) (size 1.6 1.6) (drill 0.8) (layers *.Cu *.Mask)
+      (net 3 GND))
+    (pad 2 thru_hole circle (at 5 0 270) (size 1.6 1.6) (drill 0.8) (layers *.Cu *.Mask)
+      (net 52 "Net-(C21-Pad2)"))
+    (model ${KISYS3DMOD}/Capacitors_THT.3dshapes/C_Disc_D5.0mm_W2.5mm_P5.00mm.wrl
+      (at (xyz 0 0 0))
+      (scale (xyz 1 1 1))
+      (rotate (xyz 0 0 0))
+    )
+  )
   (gr_line (start 26 106) (end 26 43) (angle 90) (layer Edge.Cuts) (width 0.15))
   (gr_line (start 266 106) (end 26 106) (angle 90) (layer Edge.Cuts) (width 0.15))
@@
   (segment (start 217 50) (end 217 45.428) (width 2) (layer F.Cu) (net 38))
   (segment (start 242 50) (end 242 51.25) (width 2) (layer F.Cu) (net 38))
-  (segment (start 242 51.25) (end 246 57) (width 2) (layer F.Cu) (net 38))
-  (segment (start 252.5 56.75) (end 260.75 65) (width 2) (layer F.Cu) (net 38))
-  (segment (start 246 57) (end 252.5 56.75) (width 2) (layer F.Cu) (net 38))
+  (segment (start 242 51.25) (end 247.5 55.5) (width 2) (layer F.Cu) (net 38))
+  (segment (start 252.75 58.5) (end 260.75 65) (width 2) (layer F.Cu) (net 38))
+  (segment (start 247.5 55.5) (end 252.75 58.5) (width 2) (layer F.Cu) (net 38))
   (segment (start 167 50) (end 167 48) (width 2) (layer B.Cu) (net 38))
   (segment (start 167 48) (end 164 44.5) (width 2) (layer B.Cu) (net 38))
@@
   (segment (start 136.25 86.125) (end 139.125 89) (width 0.5) (layer B.Cu) (net 50))
   (segment (start 136.25 82.21) (end 136.25 84.75) (width 0.5) (layer B.Cu) (net 50))
+  (segment (start 263 97.25) (end 263 103) (width 0.5) (layer B.Cu) (net 51))
+  (segment (start 29 97.5) (end 29 103) (width 0.5) (layer B.Cu) (net 52) (status 10))
   (zone (net 11) (net_name OUTPUT) (layer F.Cu) (hatch edge 0.508)
     (connect_pads (clearance 1))

Commit message: Submitted to JLCPCB 2020-08-24
Parts:
- C1: footprint Capacitors_THT:C_Axial_L5.1mm_D3.1mm_P10.00mm_Horizontal -> Capacitors_THT:C_Rect_L16.5mm_W5.0mm_P15.00mm_MKT
- D1: value 1N4477 -> 1N4752A
- moved C12 30.5 mm to (50.8, 75.0)
- moved R13 20.7 mm to (75.2, 101.8)
- moved R41 20.6 mm to (78.2, 73.8)
- moved C11 20.3 mm to (68.0, 70.0)
- moved J3 18.5 mm to (82.5, 71.8)
- moved D1 13.0 mm to (75.5, 98.0), turned to 90 degrees
- moved C8 12.9 mm to (66.8, 79.8)
- moved C7 12.8 mm to (66.8, 96.0)
- moved R15 12.8 mm to (79.5, 94.2)
- moved D5 9.75 mm to (56.8, 69.8)
- moved R2 5.94 mm to (136.2, 98.8), turned to 90 degrees
- moved C1 5.76 mm to (139.5, 93.0)
- moved C17 3.01 mm to (42.5, 90.2)
- moved R8 2.75 mm to (154.5, 99.8)
- moved Q8 2.14 mm to (110.5, 89.8), turned to 270 degrees
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Connections:
- Q8 pad 1: GND -> Net-(Q10-Pad3)
- Q8 pad 3: Net-(Q10-Pad3) -> GND
Routing:
- net Net-(C4-Pad2): track 28.8 -> 52.0 mm
- net +48V: track 302.0 -> 316.2 mm
- net Net-(C6-Pad1): track 44.4 -> 32.3 mm
- net OUTPUT: track 390.5 -> 399.2 mm
- net Net-(C1-Pad1): track 21.5 -> 12.9 mm
- net Net-(R10-Pad2): track 44.7 -> 42.2 mm
- net Net-(C7-Pad1): track 14.7 -> 13.5 mm
- net Net-(C11-Pad1): track 5.75 -> 4.88 mm
- net Net-(C20-Pad2): track 5.75 -> 5.00 mm
- net Net-(Q10-Pad3): track 36.6 -> 37.3 mm
- net Net-(C9-Pad1): track 27.3 -> 26.8 mm
- net INPUT: track 24.9 -> 25.4 mm
- net Net-(C21-Pad2): track 5.50 -> 5.00 mm

Commit message: Changed softstart and Poweramp to TO-220 transistors
Parts:
- added L1: 1 uH, Inductors_THT:L_Radial_D16.8mm_P11.43mm_Vishay_IHB-1, F.Cu at (261.0, 78.0)
- added R42: 3k3, Resistors_THT:R_Axial_DIN0411_L9.9mm_D3.6mm_P15.24mm_Horizontal, F.Cu at (241.0, 71.0)
- C9: value 33 pF -> 47 pF
- Q10, Q16: value MJE350 -> MJE15033; footprint TO_SOT_Packages_THT:TO-126_Vertical -> TO_SOT_Packages_THT:TO-220-3_Vertical
- Q11, Q12, Q15: value MJE340 -> MJE15032; footprint TO_SOT_Packages_THT:TO-126_Vertical -> TO_SOT_Packages_THT:TO-220-3_Vertical
- moved J1 26.6 mm to (245.5, 101.0)
- moved R23 6.05 mm to (153.0, 83.0)
- moved Q11 6.02 mm to (147.0, 73.5), turned to 0 degrees
- moved Q12 5.83 mm to (166.0, 77.0), turned to 180 degrees
- moved Q10 4.88 mm to (126.5, 82.0), turned to 270 degrees
- moved R21 4.51 mm to (142.0, 79.5)
- moved C10 2.79 mm to (155.0, 87.0)
- moved R22 1.77 mm to (137.5, 86.0)
- moved J2 1.52 mm to (229.5, 74.5)
Connections:
- C11 pad 2: OUTPUT -> Net-(C11-Pad2)
- C6 pad 2: OUTPUT -> Net-(C11-Pad2)
- D5 pad 2: OUTPUT -> Net-(C11-Pad2)
- D6 pad 1: OUTPUT -> Net-(C11-Pad2)
- Q11 pad 1: Net-(C10-Pad1) -> Net-(Q11-Pad1)
- Q11 pad 3: Net-(Q11-Pad3) -> Net-(C10-Pad1)
- Q12 pad 1: Net-(Q12-Pad1) -> Net-(C5-Pad2)
- Q12 pad 3: Net-(C5-Pad2) -> Net-(Q12-Pad3)
- Q13 pad 3: OUTPUT -> Net-(C11-Pad2)
- Q14 pad 3: OUTPUT -> Net-(C11-Pad2)
- Q15 pad 1: Net-(Q15-Pad1) -> Net-(C10-Pad2)
- Q15 pad 3: Net-(C10-Pad2) -> Net-(Q15-Pad3)
- Q16 pad 1: Net-(Q16-Pad1) -> Net-(C10-Pad1)
- Q16 pad 3: Net-(C10-Pad1) -> Net-(Q16-Pad3)
- Q17 pad 1: Net-(Q15-Pad1) -> Net-(Q15-Pad3)
- Q18 pad 1: Net-(Q16-Pad1) -> Net-(Q16-Pad3)
- Q19 pad 1: Net-(Q15-Pad1) -> Net-(Q15-Pad3)
- Q20 pad 1: Net-(Q16-Pad1) -> Net-(Q16-Pad3)
- Q21 pad 1: Net-(Q15-Pad1) -> Net-(Q15-Pad3)
- Q22 pad 1: Net-(Q16-Pad1) -> Net-(Q16-Pad3)
- Q23 pad 1: Net-(Q15-Pad1) -> Net-(Q15-Pad3)
- Q24 pad 1: Net-(Q16-Pad1) -> Net-(Q16-Pad3)
- Q8 pad 1: Net-(Q10-Pad3) -> Net-(Q10-Pad1)
- Q9 pad 1: Net-(Q10-Pad3) -> Net-(Q10-Pad1)
- R14 pad 1: OUTPUT -> Net-(C11-Pad2)
- R17 pad 1: Net-(Q10-Pad3) -> Net-(Q10-Pad1)
- R20 pad 1: Net-(Q10-Pad1) -> Net-(Q10-Pad3)
- R21 pad 1: Net-(Q11-Pad3) -> Net-(Q11-Pad1)
- R22 pad 3: Net-(Q11-Pad3) -> Net-(Q11-Pad1)
- R24 pad 2: Net-(Q12-Pad1) -> Net-(Q12-Pad3)
- R26 pad 2: OUTPUT -> Net-(C11-Pad2)
- R27 pad 1: OUTPUT -> Net-(C11-Pad2)
- R31 pad 1: OUTPUT -> Net-(C11-Pad2)
- R31 pad 2: Net-(Q15-Pad1) -> Net-(Q15-Pad3)
- R32 pad 1: Net-(Q16-Pad1) -> Net-(Q16-Pad3)
- R32 pad 2: OUTPUT -> Net-(C11-Pad2)
- R33 pad 1: OUTPUT -> Net-(C11-Pad2)
- R34 pad 2: OUTPUT -> Net-(C11-Pad2)
- R35 pad 1: OUTPUT -> Net-(C11-Pad2)
- R36 pad 2: OUTPUT -> Net-(C11-Pad2)
- R37 pad 1: OUTPUT -> Net-(C11-Pad2)
- R38 pad 2: OUTPUT -> Net-(C11-Pad2)
- R39 pad 1: OUTPUT -> Net-(C11-Pad2)
- R40 pad 2: OUTPUT -> Net-(C11-Pad2)
Routing:
- net Net-(C11-Pad2): track 0.00 -> 405.9 mm
- net OUTPUT: track 399.2 -> 40.7 mm
- net Net-(Q15-Pad1): track 160.6 -> 0.00 mm
- net Net-(Q15-Pad3): track 0.00 -> 159.5 mm
- net Net-(Q16-Pad1): track 159.4 -> 0.00 mm
- net Net-(Q16-Pad3): track 0.00 -> 153.8 mm
- net Net-(Q10-Pad1): track 10.7 -> 38.0 mm
- net Net-(Q10-Pad3): track 37.3 -> 10.8 mm
- net Net-(Q11-Pad3): track 15.2 -> 0.00 mm
- net Net-(Q12-Pad1): track 14.8 -> 0.00 mm
- net Net-(Q12-Pad3): track 0.00 -> 14.6 mm
- net Net-(Q11-Pad1): track 0.00 -> 14.6 mm
- net Net-(C10-Pad2): track 86.1 -> 89.5 mm
- net Net-(R22-Pad1): track 13.5 -> 11.1 mm
- net Net-(C10-Pad1): track 64.5 -> 62.8 mm
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