File: PowerampC300MJE340350/PowerampC300.sch (KiCad schematic (older format))
At the start: 109 parts, among them J1 Conn_01x02, J2 Conn_01x02, J3 Conn_01x02, J4 Conn_01x01, J5 Conn_01x01, J6 Conn_01x01, J7 Conn_01x01, J8 Conn_01x02, J9 Conn_Coaxial, Q1 2N5551, Q10 MJE350, Q11 MJE340, Q12 MJE340, Q13 2N5551, Q14 2N5401, Q15 MJE340, Q16 MJE350, Q17 MJL3281A, Q18 MJL1302A, Q19 MJL3281A, Q2 2N5551, Q20 MJL1302A, Q21 MJL3281A, Q22 MJL1302A, Q23 MJL3281A, Q24 MJL1302A, Q3 2N5401, Q4 2N5401, Q5 2N5551, Q6 2N5551, Q7 2N5551, Q8 2N5401, Q9 2N5401

Commit message: Working design 2020-10-12
Parts:
- removed Q9: 2N5401, TO_SOT_Packages_THT:TO-92_Inline_Wide, symbol Q_PNP_EBC
- removed R18: 330R, Resistors_THT:R_Axial_DIN0207_L6.3mm_D2.5mm_P7.62mm_Horizontal, symbol R
- removed R20: 27R, Resistors_THT:R_Axial_DIN0207_L6.3mm_D2.5mm_P7.62mm_Horizontal, symbol R
- added R43: 10k, Resistors_THT:R_Axial_DIN0309_L9.0mm_D3.2mm_P12.70mm_Horizontal, symbol R
- R19: value 10R -> 33R; footprint Resistors_THT:R_Axial_DIN0207_L6.3mm_D2.5mm_P7.62mm_Horizontal -> Resistors_THT:R_Axial_DIN0309_L9.0mm_D3.2mm_P12.70mm_Horizontal; LCSC C176452 -> C176446
- R23: value 150R -> 100R
Connections:
- net GND: now also R43.1
- net at C6.2, D5.2 (A), D6.1 (K)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: now also R43.2
- net at R19.1: now also Q10.1 (E)
Other:
- moved on the sheet: J2, L1, Q10, R42
Changed lines of the file:
@@
 P 3900 4900
 F 0 "R23" V 3980 4900 50  0000 C CNN
-F 1 "150R" V 3900 4900 50  0000 C CNN
+F 1 "100R" V 3900 4900 50  0000 C CNN
 F 2 "Resistors_THT:R_Axial_DIN0207_L6.3mm_D2.5mm_P7.62mm_Horizontal" V 3830 4900 50  0001 C CNN
 F 3 "" H 3900 4900 50  0001 C CNN
@@
 F 4 "C57435" V 3100 2050 60  0001 C CNN "LCSC"
 	1    3100 2050
-	-1   0    0    1
-$EndComp
-$Comp
-L R R18
-U 1 1 5F3B6B8B
-P 3500 1950
-F 0 "R18" V 3580 1950 50  0000 C CNN
-F 1 "330R" V 3500 1950 50  0000 C CNN
-F 2 "Resistors_THT:R_Axial_DIN0207_L6.3mm_D2.5mm_P7.62mm_Horizontal" V 3430 1950 50  0001 C CNN
-F 3 "" H 3500 1950 50  0001 C CNN
-F 4 "C58608" V 3500 1950 60  0001 C CNN "LCSC"
-	1    3500 1950
-	-1   0    0    1
-$EndComp
-$Comp
-L R R19
-U 1 1 5F3B6E0F
-P 3900 2050
-F 0 "R19" V 3980 2050 50  0000 C CNN
-F 1 "10R" V 3900 2050 50  0000 C CNN
-F 2 "Resistors_THT:R_Axial_DIN0207_L6.3mm_D2.5mm_P7.62mm_Horizontal" V 3830 2050 50  0001 C CNN
-F 3 "" H 3900 2050 50  0001 C CNN
-F 4 "C176452" V 3900 2050 60  0001 C CNN "LCSC"
-	1    3900 2050
-	-1   0    0    1
-$EndComp
-$Comp
-L R R20
-U 1 1 5F3B7026
-P 3900 2600
-F 0 "R20" V 3980 2600 50  0000 C CNN
-F 1 "27R" V 3900 2600 50  0000 C CNN
-F 2 "Resistors_THT:R_Axial_DIN0207_L6.3mm_D2.5mm_P7.62mm_Horizontal" V 3830 2600 50  0001 C CNN
-F 3 "" H 3900 2600 50  0001 C CNN
-F 4 "C176487" V 3900 2600 60  0001 C CNN "LCSC"
-	1    3900 2600
 	-1   0    0    1
 $EndComp
@@
 	1    0    0    -1
 $EndComp
-Text GLabel 10450 4200 2    60   Input ~ 0
+Text GLabel 10700 4200 2    60   Input ~ 0
 OUTPUT
 Text GLabel 650  3900 3    60   Input ~ 0
@@
 	-1   0    0    1
 $EndComp
-Text GLabel 10450 3600 3    60   Input ~ 0
+Text GLabel 10450 3450 3    60   Input ~ 0
 OUTPUT
 $Comp
@@
 L GND #PWR012
 U 1 1 5F3D76F6
-P 10800 4900
-F 0 "#PWR012" H 10800 4650 50  0001 C CNN
-F 1 "GND" H 10800 4750 50  0000 C CNN
-F 2 "" H 10800 4900 50  0001 C CNN
-F 3 "" H 10800 4900 50  0001 C CNN
-	1    10800 4900
+P 10850 5200
+F 0 "#PWR012" H 10850 4950 50  0001 C CNN
+F 1 "GND" H 10850 5050 50  0000 C CNN
+F 2 "" H 10850 5200 50  0001 C CNN
+F 3 "" H 10850 5200 50  0001 C CNN
+	1    10850 5200
 	1    0    0    -1
 $EndComp
 Text GLabel 10500 5900 3    60   Input ~ 0
 +48V
-Text GLabel 10550 4950 3    60   Input ~ 0
+Text GLabel 10600 5250 3    60   Input ~ 0
 -48V
 $Comp
 L Conn_01x02 J2
 U 1 1 5F3DAA81
-P 9800 4850
-F 0 "J2" H 9800 4950 50  0000 C CNN
-F 1 "Conn_01x02" H 9800 4650 50  0000 C CNN
-F 2 "Connectors_Terminal_Blocks:TerminalBlock_bornier-2_P5.08mm" H 9800 4850 50  0001 C CNN
-F 3 "" H 9800 4850 50  0001 C CNN
-F 4 "C395849" H 9800 4850 60  0001 C CNN "LCSC"
-	1    9800 4850
+P 9850 5150
+F 0 "J2" H 9850 5250 50  0000 C CNN
+F 1 "Conn_01x02" H 9850 4950 50  0000 C CNN
+F 2 "Connectors_Terminal_Blocks:TerminalBlock_bornier-2_P5.08mm" H 9850 5150 50  0001 C CNN
+F 3 "" H 9850 5150 50  0001 C CNN
+F 4 "C395849" H 9850 5150 60  0001 C CNN "LCSC"
+	1    9850 5150
 	-1   0    0    1
 $EndComp
@@
 	3100 1800 3100 1900
 Connection ~ 2600 1800
-Wire Wire Line
-	3250 2450 3250 2650
-Wire Wire Line
-	3250 2450 3100 2450
 Connection ~ 3100 2450
 Connection ~ 3100 1800
 Wire Wire Line
-	3500 2100 3500 2150
-Wire Wire Line
-	3900 2200 3900 2450
-Wire Wire Line
-	3900 2350 3800 2350
-Wire Wire Line
-	3900 1800 3900 1900
-Connection ~ 3500 1800
-Connection ~ 3900 2350
-Wire Wire Line
-	3900 2750 3900 2800
-Wire Wire Line
-	3500 2550 3500 3000
-Wire Wire Line
-	3500 3000 3600 3000
+	3900 2650 3900 3350
 Wire Wire Line
 	3700 3200 5950 3200
 Wire Wire Line
 	2750 3200 3500 3200
-Wire Wire Line
-	3900 3200 3900 3350
 Wire Wire Line
 	8950 6150 2250 6150
@@
 	5100 4050 5100 4350
 Wire Wire Line
-	3500 4200 9650 4200
+	3500 4200 10150 4200
 Connection ~ 5100 4200
 Connection ~ 3500 3700
@@
 Wire Wire Line
 	5550 1800 5550 3350
-Connection ~ 3900 1800
 Connection ~ 5100 3200
 Connection ~ 5100 5150
@@
 Connection ~ 2750 2700
 Wire Wire Line
-	3250 2650 3500 2650
-Connection ~ 3500 2650
-Wire Wire Line
 	2600 3500 2600 3300
 Connection ~ 6250 1800
@@
 	10050 5700 10650 5700
 Wire Wire Line
-	10550 4950 10550 4850
-Wire Wire Line
-	10550 4850 10000 4850
-Wire Wire Line
-	10000 4750 10800 4750
+	10600 5250 10600 5150
+Wire Wire Line
+	10600 5150 10050 5150
+Wire Wire Line
+	10050 5050 10850 5050
 Wire Wire Line
 	10050 5800 10500 5800
@@
 	4750 4100 4200 4100
 Connection ~ 4200 4100
-Wire Wire Line
-	10450 3450 10450 3600
 Wire Wire Line
 	9900 3350 10700 3350
@@
 Connection ~ 8900 2350
 Wire Wire Line
-	9450 3950 9450 4250
+	9450 4200 9450 4250
 Connection ~ 9450 4200
 Connection ~ 9150 5600
@@
 Connection ~ 8750 1100
 Wire Wire Line
-	10800 4750 10800 4900
+	10850 5050 10850 5200
 $Comp
 L L L1
 U 1 1 5F55AD15
-P 9800 4200
-F 0 "L1" V 9750 4200 50  0000 C CNN
-F 1 "1 uH" V 9875 4200 50  0000 C CNN
-F 2 "Inductors_THT:L_Radial_D16.8mm_P11.43mm_Vishay_IHB-1" H 9800 4200 50  0001 C CNN
-F 3 "" H 9800 4200 50  0001 C CNN
-	1    9800 4200
+P 10300 4200
+F 0 "L1" V 10250 4200 50  0000 C CNN
+F 1 "1 uH" V 10375 4200 50  0000 C CNN
+F 2 "Inductors_THT:L_Radial_D16.8mm_P11.43mm_Vishay_IHB-1" H 10300 4200 50  0001 C CNN
+F 3 "" H 10300 4200 50  0001 C CNN
+	1    10300 4200
 	0    1    1    0
 $EndComp
@@
 L R R42
 U 1 1 5F55B21A
-P 9800 3950
-F 0 "R42" V 9880 3950 50  0000 C CNN
-F 1 "4R7" V 9800 3950 50  0000 C CNN
-F 2 "Resistors_THT:R_Axial_DIN0411_L9.9mm_D3.6mm_P15.24mm_Horizontal" V 9730 3950 50  0001 C CNN
-F 3 "" H 9800 3950 50  0001 C CNN
-F 4 "C138189" V 9800 3950 60  0001 C CNN "LCSC"
-	1    9800 3950
+P 10300 3950
+F 0 "R42" V 10380 3950 50  0000 C CNN
+F 1 "4R7" V 10300 3950 50  0000 C CNN
+F 2 "Resistors_THT:R_Axial_DIN0411_L9.9mm_D3.6mm_P15.24mm_Horizontal" V 10230 3950 50  0001 C CNN
+F 3 "" H 10300 3950 50  0001 C CNN
+F 4 "C138189" V 10300 3950 60  0001 C CNN "LCSC"
+	1    10300 3950
 	0    -1   -1   0
 $EndComp
 Wire Wire Line
-	9650 3950 9450 3950
-Wire Wire Line
-	9950 3950 10100 3950
-Wire Wire Line
-	10100 3950 10100 4200
-Wire Wire Line
-	9950 4200 10450 4200
-Connection ~ 10100 4200
+	10450 3950 10600 3950
+Wire Wire Line
+	10600 3950 10600 4200
+Wire Wire Line
+	10450 4200 10700 4200
+Connection ~ 10600 4200
 $Comp
 L Q_NPN_EBC Q5
@@
 $EndComp
 $Comp
-L Q_PNP_EBC Q9
-U 1 1 5F5DBD1F
-P 3600 2350
-F 0 "Q9" H 3800 2400 50  0000 L CNN
-F 1 "2N5401" H 3800 2300 50  0000 L CNN
-F 2 "TO_SOT_Packages_THT:TO-92_Inline_Wide" H 3800 2450 50  0001 C CNN
-F 3 "" H 3600 2350 50  0001 C CNN
-	1    3600 2350
-	-1   0    0    1
-$EndComp
-$Comp
 L Q_NPN_EBC Q6
 U 1 1 5F5DC924
@@
 $EndComp
 Connection ~ 9100 1800
-Connection ~ 8800 1800
 Connection ~ 9150 5000
 Wire Wire Line
@@
 L Q_PNP_ECB Q10
 U 1 1 5F686C2D
-P 3800 3000
-F 0 "Q10" H 4000 3050 50  0000 L CNN
-F 1 "MJE350" H 4000 2950 50  0000 L CNN
-F 2 "TO_SOT_Packages_THT:TO-126_Vertical" H 4000 3100 50  0001 C CNN
-F 3 "" H 3800 3000 50  0001 C CNN
-	1    3800 3000
+P 3800 2450
+F 0 "Q10" H 4000 2500 50  0000 L CNN
+F 1 "MJE350" H 4000 2400 50  0000 L CNN
+F 2 "TO_SOT_Packages_THT:TO-126_Vertical" H 4000 2550 50  0001 C CNN
+F 3 "" H 3800 2450 50  0001 C CNN
+	1    3800 2450
 	1    0    0    1
 $EndComp
@@
 	1    0    0    1
 $EndComp
+Wire Wire Line
+	10150 3950 10050 3950
+Wire Wire Line
+	10050 3950 10050 4200
+Connection ~ 10050 4200
+$Comp
+L R R43
+U 1 1 5F838DE0
+P 9850 4400
+F 0 "R43" V 9930 4400 50  0000 C CNN
+F 1 "10k" V 9850 4400 50  0000 C CNN
+F 2 "Resistors_THT:R_Axial_DIN0309_L9.0mm_D3.2mm_P12.70mm_Horizontal" V 9780 4400 50  0001 C CNN
+F 3 "" H 9850 4400 50  0001 C CNN
+F 4 "C57725" V 9850 4400 60  0001 C CNN "LCSC"
+	1    9850 4400
+	1    0    0    1
+$EndComp
+$Comp
+L GND #PWR017
+U 1 1 5F838F45
+P 9850 4600
+F 0 "#PWR017" H 9850 4350 50  0001 C CNN
+F 1 "GND" H 9850 4450 50  0000 C CNN
+F 2 "" H 9850 4600 50  0001 C CNN
+F 3 "" H 9850 4600 50  0001 C CNN
+	1    9850 4600
+	1    0    0    -1
+$EndComp
+Wire Wire Line
+	9850 4600 9850 4550
+Wire Wire Line
+	9850 4250 9850 4200
+Connection ~ 9850 4200
+Wire Wire Line
+	3900 1900 3900 1800
+Connection ~ 3900 1800
+Wire Wire Line
+	3900 2200 3900 2250
+Wire Wire Line
+	3600 2450 3100 2450
+$Comp
+L R R19
+U 1 1 5F8495EB
+P 3900 2050
+F 0 "R19" V 3980 2050 50  0000 C CNN
+F 1 "33R" V 3900 2050 50  0000 C CNN
+F 2 "Resistors_THT:R_Axial_DIN0309_L9.0mm_D3.2mm_P12.70mm_Horizontal" V 3830 2050 50  0001 C CNN
+F 3 "" H 3900 2050 50  0001 C CNN
+F 4 "C176446" V 3900 2050 60  0001 C CNN "LCSC"
+	1    3900 2050
+	-1   0    0    1
+$EndComp
 $EndSCHEMATC

Commit message: Changed grounding and star layout
Parts:
- removed C20, C21: 0.1 uF, Capacitors_THT:C_Disc_D5.0mm_W2.5mm_P5.00mm, symbol C_Small
- added C24: SHORT, Capacitors_THT:C_Disc_D5.0mm_W2.5mm_P5.00mm, symbol C_Small
- added C25: 0.1 uF, Capacitors_THT:C_Axial_L3.8mm_D2.6mm_P10.00mm_Horizontal, symbol C_Small
- added JP1, JP2: Jumper_NO_Small, Pin_Headers:Pin_Header_Straight_1x02_Pitch2.54mm, symbol Jumper_NO_Small
- added R18: NC, Resistors_THT:R_Axial_DIN0207_L6.3mm_D2.5mm_P7.62mm_Horizontal, symbol R
- C3: value 220 pF -> 150 pF
- C9: value 100 pF -> 150 pF
Connections:
- net GND: now also C25.2, JP1.1, JP2.1
- net at C10.2, D3.2 (A), Q10.2 (C)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: now also C24.2; no longer C9.2
- net at J4.1 (Pin_1): now also JP1.2
- net at J6.1 (Pin_1): now also JP2.2
- new net: C24.1, C9.2, R18.1
- new net: C25.1, R18.2
Other:
- moved on the sheet: C9
