File: PowerampC300TO126/PowerampC300.kicad_pcb (KiCad board)
At the start: 2 copper layers, 240 x 63 mm, 110 parts, among them J1 Conn_01x02, J2 Conn_01x02, J3 Conn_01x02, J4 Conn_01x01, J5 Conn_01x01, J6 Conn_01x01, J7 Conn_01x01, J8 Conn_01x02, J9 Conn_Coaxial, Q1 2N5551, Q10 MJE350, Q11 MJE340, Q12 MJE340, Q13 2N5551, Q14 2N5401, Q15 MJE340, Q16 MJE350, Q17 MJL3281A, Q18 MJL1302A, Q19 MJL3281A, Q2 2N5551, Q20 MJL1302A, Q21 MJL3281A, Q22 MJL1302A, Q23 MJL3281A, Q24 MJL1302A, Q3 2N5401, Q4 2N5401, Q5 2N5551, Q6 2N5551, Q7 2N5551, Q8 2N5401

Commit message: Moved Q1 and Q2 together
Parts:
- C24: value SHORT -> 0.1 uF; footprint Capacitors_THT:C_Disc_D5.0mm_W2.5mm_P5.00mm -> Capacitors_THT:C_Axial_L3.8mm_D2.6mm_P10.00mm_Horizontal
- C25: value 0.1 uF -> SHORT; footprint Capacitors_THT:C_Axial_L3.8mm_D2.6mm_P10.00mm_Horizontal -> Capacitors_THT:C_Disc_D5.0mm_W2.5mm_P5.00mm
- R5: value 620R -> 1k
- moved D1 18.5 mm to (52.8, 103.0), turned to 180 degrees
- moved C25 13.0 mm to (134.9, 93.0)
- moved C24 13.0 mm to (121.6, 92.8)
- moved Q2 10.3 mm to (120.0, 102.8), turned to 180 degrees
- moved Q8 9.90 mm to (107.2, 98.8), turned to 180 degrees
- moved C9 8.04 mm to (103.0, 93.6)
- moved Q1 7.00 mm to (114.8, 98.8), turned to 0 degrees
- moved C6 5.23 mm to (74.0, 104.2)
- moved C4 5.11 mm to (69.2, 104.2)
- moved R15 4.41 mm to (79.0, 96.8)
- moved Q5 4.35 mm to (97.0, 101.6)
- moved R14 4.22 mm to (82.8, 96.6)
- moved C8 3.71 mm to (72.8, 94.4)
- moved Q6 3.60 mm to (89.4, 101.6)
- moved R2 3.22 mm to (164.2, 95.4)
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Connections:
- C24 pad 2: Net-(C10-Pad2) -> GND
- C25 pad 2: GND -> Net-(C10-Pad2)
- C9 pad 2: Net-(C24-Pad1) -> Net-(C25-Pad1)
- R18 pad 1: Net-(C24-Pad1) -> Net-(C25-Pad1)
- R18 pad 2: Net-(C25-Pad1) -> Net-(C24-Pad1)
Routing:
- net Net-(C24-Pad1): track 31.3 -> 3.17 mm
- net Net-(C25-Pad1): track 2.92 -> 30.0 mm
- net Net-(C6-Pad1): track 34.3 -> 48.5 mm
- net +48V: track 297.2 -> 308.6 mm
- net Net-(Q2-Pad1): track 18.7 -> 7.99 mm
- net Net-(C10-Pad2): track 83.3 -> 91.0 mm
- net Net-(Q1-Pad1): track 6.66 -> 13.9 mm
- net Net-(C10-Pad1): track 63.9 -> 70.8 mm
- net Net-(C2-Pad2): track 28.2 -> 35.0 mm
- net Net-(Q10-Pad3): track 44.2 -> 50.8 mm
- net Net-(Q1-Pad3): track 22.8 -> 29.3 mm
- net Net-(C1-Pad1): track 13.5 -> 19.9 mm
- net Net-(Q2-Pad3): track 20.6 -> 26.8 mm
- net Net-(C3-Pad2): track 35.1 -> 41.2 mm
- net GND: track 57.5 -> 52.5 mm
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