File: PowerampC300TO126/PowerampC300.sch (KiCad schematic (older format))
At the start: 127 parts, among them J1 Conn_01x02, J2 Conn_01x02, J3 Conn_01x02, J4 Conn_01x01, J5 Conn_01x01, J6 Conn_01x01, J7 Conn_01x01, J8 Conn_01x02, J9 Conn_Coaxial, Q1 2N5551, Q10 MJE350, Q11 MJE340, Q12 MJE340, Q13 2N5551, Q14 2N5401, Q15 MJE340, Q16 MJE350, Q17 MJL3281A, Q18 MJL1302A, Q19 MJL3281A, Q2 2N5551, Q20 MJL1302A, Q21 MJL3281A, Q22 MJL1302A, Q23 MJL3281A, Q24 MJL1302A, Q3 2N5401, Q4 2N5401, Q5 2N5551, Q6 2N5551, Q7 2N5551, Q8 2N5401, U1 MOC3020M

Commit message: Added back Q9 transistor for Q8 protection
Parts:
- added Q9: 2N5401, TO_SOT_Packages_THT:TO-92_Inline_Wide, symbol Q_PNP_EBC
Connections:
- net +48V: now also Q9.1 (E)
- net at C20.1, C9.1, Q3.3 (C)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: now also Q9.3 (C)
- net at Q10.1 (E), R19.1: now also Q9.2 (B)
Changed lines of the file:
@@
 Connection ~ 6250 3450
 Wire Wire Line
-	2750 2700 2750 3200
+	2750 2400 2750 3200
 Wire Wire Line
 	2600 3500 2600 3300
@@
 Wire Wire Line
 	9500 4100 9450 4100
+$Comp
+L Q_PNP_EBC Q9
+U 1 1 60A7449B
+P 3650 2200
+F 0 "Q9" H 3850 2250 50  0000 L CNN
+F 1 "2N5401" H 3850 2150 50  0000 L CNN
+F 2 "TO_SOT_Packages_THT:TO-92_Inline_Wide" H 3850 2300 50  0001 C CNN
+F 3 "" H 3650 2200 50  0001 C CNN
+	1    3650 2200
+	-1   0    0    1
+$EndComp
+Wire Wire Line
+	3900 2200 3850 2200
+Wire Wire Line
+	3550 2000 3550 1800
+Connection ~ 3550 1800
+Wire Wire Line
+	3550 2400 2750 2400
+Connection ~ 2750 2700
 $EndSCHEMATC
