File: PowerCond/PowerCond.sch (KiCad schematic (older format))
At the start: 62 parts, among them J1 Conn_01x02, J10 Conn_01x01, J11 Conn_01x01, J12 Conn_01x01, J2 Conn_01x02, J3 Conn_01x02, J4 Conn_01x02, J5 Conn_01x02, J6 Conn_01x02, J7 Conn_01x02, J8 Conn_01x02, J9 Conn_01x01, T1 Transformer_1P1Sdotted, T2 Transformer_1P1Sdotted, T3 Transformer_1P1Sdotted, T4 Transformer_1P1Sdotted

Commit message: Added option for spade terminal power connections
Parts:
- J1, J2, J3, J4, J5, J6, J7, J8: footprint Connectors_Terminal_Blocks:TerminalBlock_bornier-2_P5.08mm -> PowerCond:TerminalBlock_bornier-2_P5.08mm_with_spade
Changed lines of the file:
@@
 F 0 "J2" H 1750 3250 50  0000 C CNN
 F 1 "Conn_01x02" H 1800 3350 50  0000 C CNN
-F 2 "Connectors_Terminal_Blocks:TerminalBlock_bornier-2_P5.08mm" H 1750 3150 50  0001 C CNN
+F 2 "PowerCond:TerminalBlock_bornier-2_P5.08mm_with_spade" H 1750 3150 50  0001 C CNN
 F 3 "" H 1750 3150 50  0001 C CNN
 F 4 "C395849" H 1750 3150 60  0001 C CNN "LCSC"
@@
 F 0 "J3" H 1750 4050 50  0000 C CNN
 F 1 "Conn_01x02" H 1750 3750 50  0000 C CNN
-F 2 "Connectors_Terminal_Blocks:TerminalBlock_bornier-2_P5.08mm" H 1750 3950 50  0001 C CNN
+F 2 "PowerCond:TerminalBlock_bornier-2_P5.08mm_with_spade" H 1750 3950 50  0001 C CNN
 F 3 "" H 1750 3950 50  0001 C CNN
 F 4 "C395849" H 1750 3950 60  0001 C CNN "LCSC"
@@
 F 0 "J1" H 1750 2800 50  0000 C CNN
 F 1 "Conn_01x02" H 1750 2500 50  0000 C CNN
-F 2 "Connectors_Terminal_Blocks:TerminalBlock_bornier-2_P5.08mm" H 1750 2700 50  0001 C CNN
+F 2 "PowerCond:TerminalBlock_bornier-2_P5.08mm_with_spade" H 1750 2700 50  0001 C CNN
 F 3 "" H 1750 2700 50  0001 C CNN
 F 4 "C395849" H 1750 2700 60  0001 C CNN "LCSC"
@@
 F 0 "J4" H 1750 4500 50  0000 C CNN
 F 1 "Conn_01x02" H 1750 4200 50  0000 C CNN
-F 2 "Connectors_Terminal_Blocks:TerminalBlock_bornier-2_P5.08mm" H 1750 4400 50  0001 C CNN
+F 2 "PowerCond:TerminalBlock_bornier-2_P5.08mm_with_spade" H 1750 4400 50  0001 C CNN
 F 3 "" H 1750 4400 50  0001 C CNN
 F 4 "C395849" H 1750 4400 60  0001 C CNN "LCSC"
@@
 F 0 "J5" H 8500 3050 50  0000 C CNN
 F 1 "Conn_01x02" H 8500 2750 50  0000 C CNN
-F 2 "Connectors_Terminal_Blocks:TerminalBlock_bornier-2_P5.08mm" H 8500 2950 50  0001 C CNN
+F 2 "PowerCond:TerminalBlock_bornier-2_P5.08mm_with_spade" H 8500 2950 50  0001 C CNN
 F 3 "" H 8500 2950 50  0001 C CNN
 F 4 "C395849" H 8500 2950 60  0001 C CNN "LCSC"
@@
 F 0 "J6" H 8500 4000 50  0000 C CNN
 F 1 "Conn_01x02" H 8500 3700 50  0000 C CNN
-F 2 "Connectors_Terminal_Blocks:TerminalBlock_bornier-2_P5.08mm" H 8500 3900 50  0001 C CNN
+F 2 "PowerCond:TerminalBlock_bornier-2_P5.08mm_with_spade" H 8500 3900 50  0001 C CNN
 F 3 "" H 8500 3900 50  0001 C CNN
 F 4 "C395849" H 8500 3900 60  0001 C CNN "LCSC"
@@
 F 0 "J7" H 8900 3050 50  0000 C CNN
 F 1 "Conn_01x02" H 8900 2750 50  0000 C CNN
-F 2 "Connectors_Terminal_Blocks:TerminalBlock_bornier-2_P5.08mm" H 8900 2950 50  0001 C CNN
+F 2 "PowerCond:TerminalBlock_bornier-2_P5.08mm_with_spade" H 8900 2950 50  0001 C CNN
 F 3 "" H 8900 2950 50  0001 C CNN
 F 4 "C395849" H 8900 2950 60  0001 C CNN "LCSC"
@@
 F 0 "J8" H 8900 4000 50  0000 C CNN
 F 1 "Conn_01x02" H 8900 3700 50  0000 C CNN
-F 2 "Connectors_Terminal_Blocks:TerminalBlock_bornier-2_P5.08mm" H 8900 3900 50  0001 C CNN
+F 2 "PowerCond:TerminalBlock_bornier-2_P5.08mm_with_spade" H 8900 3900 50  0001 C CNN
 F 3 "" H 8900 3900 50  0001 C CNN
 F 4 "C395849" H 8900 3900 60  0001 C CNN "LCSC"
