File: PowerampSimpleParts/PowerampC300.sch (KiCad schematic (older format))
At the start: 121 parts, among them J1 Conn_01x02, J2 Conn_01x02, J3 Conn_01x02, J4 Conn_01x01, J5 Conn_01x01, J6 Conn_01x01, J7 Conn_01x01, J8 Conn_01x02, J9 Conn_Coaxial, Q1 2N5551, Q10 2N5401, Q11 TIP41C, Q12 2N5551, Q13 2N5551, Q14 2N5401, Q15 TIP41C, Q16 TIP42C, Q17 TIP41C, Q18 TIP42C, Q19 TIP41C, Q2 2N5551, Q20 TIP42C, Q21 TIP41C, Q22 TIP42C, Q23 TIP41C, Q24 TIP42C, Q25 2N5551, Q26 2N5401, Q3 2N5401, Q4 2N5401, Q5 2N5551, Q6 2N5551, Q7 2N5551, Q8 2N5401, Q9 2N5401

Commit message: A few minor tweaks to PowerampSimpleParts layout
Parts:
- removed R31: 33R, Resistors_THT:R_Axial_DIN0411_L9.9mm_D3.6mm_P12.70mm_Horizontal, symbol R
- removed R52: 100R, Resistors_THT:R_Axial_DIN0207_L6.3mm_D2.5mm_P7.62mm_Horizontal, symbol R
- added C16: NC, Capacitors_THT:C_Disc_D5.0mm_W2.5mm_P5.00mm, symbol C_Small
- R32: value 33R -> 150R
Connections:
- net BIAS1: now also C16.2
- net GND: now also C16.1
- net at Q15.3 (E), R44.1, R45.1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: now also R32.2
Other:
- moved on the sheet: R32
Changed lines of the file:
@@
-$EndComp
-$Comp
-L R R31
-U 1 1 5F3BCB79
-P 6250 3650
-F 0 "R31" V 6330 3650 50  0000 C CNN
-F 1 "33R" V 6250 3650 50  0000 C CNN
-F 2 "Resistors_THT:R_Axial_DIN0411_L9.9mm_D3.6mm_P12.70mm_Horizontal" V 6180 3650 50  0001 C CNN
-F 3 "" H 6250 3650 50  0001 C CNN
-F 4 "C173006" V 6250 3650 60  0001 C CNN "LCSC"
-	1    6250 3650
-	-1   0    0    1
 $EndComp
 $Comp
 L R R32
 U 1 1 5F3BDA9D
-P 6250 4750
-F 0 "R32" V 6330 4750 50  0000 C CNN
-F 1 "33R" V 6250 4750 50  0000 C CNN
-F 2 "Resistors_THT:R_Axial_DIN0411_L9.9mm_D3.6mm_P12.70mm_Horizontal" V 6180 4750 50  0001 C CNN
-F 3 "" H 6250 4750 50  0001 C CNN
-F 4 "C173006" V 6250 4750 60  0001 C CNN "LCSC"
-	1    6250 4750
+P 6250 4200
+F 0 "R32" V 6330 4200 50  0000 C CNN
+F 1 "150R" V 6250 4200 50  0000 C CNN
+F 2 "Resistors_THT:R_Axial_DIN0411_L9.9mm_D3.6mm_P12.70mm_Horizontal" V 6180 4200 50  0001 C CNN
+F 3 "" H 6250 4200 50  0001 C CNN
+F 4 "C173006" V 6250 4200 60  0001 C CNN "LCSC"
+	1    6250 4200
 	-1   0    0    1
 $EndComp
@@
 Connection ~ 3900 5150
 Wire Wire Line
-	5100 2750 5100 3300
+	5100 2900 5100 3300
 Connection ~ 4200 3200
 Wire Wire Line
@@
 Connection ~ 5550 6150
 Wire Wire Line
-	6250 3400 6250 3500
-Wire Wire Line
-	6250 4900 6250 4950
+	6250 3400 6250 4050
+Wire Wire Line
+	6250 4350 6250 4950
 Connection ~ 5550 4200
 Wire Wire Line
@@
 	1000 4050 1250 4050
 Wire Wire Line
-	1250 4400 1250 4050
+	1250 4050 1250 4400
 Wire Wire Line
 	1250 4700 1250 4850
 Wire Wire Line
-	750  4400 1250 4400
+	1250 4400 750  4400
 Wire Wire Line
 	750  4700 1250 4700
@@
 Connection ~ 1900 2650
 Wire Wire Line
-	4900 3550 4900 3200
+	4900 2900 4900 3550
 Connection ~ 4900 3200
 Wire Wire Line
@@
 	4900 5150 4950 5150
 Connection ~ 4950 5150
-Text GLabel 5100 2750 1    60   Input ~ 0
+Text GLabel 5100 2900 1    60   Input ~ 0
 BIAS1
 Text GLabel 5100 5550 3    60   Input ~ 0
@@
 $EndComp
 $Comp
-L R R52
-U 1 1 60D52F3E
-P 6250 4200
-F 0 "R52" V 6330 4200 50  0000 C CNN
-F 1 "100R" V 6250 4200 50  0000 C CNN
-F 2 "Resistors_THT:R_Axial_DIN0207_L6.3mm_D2.5mm_P7.62mm_Horizontal" V 6180 4200 50  0001 C CNN
-F 3 "" H 6250 4200 50  0001 C CNN
-F 4 "C172973" V 6250 4200 60  0001 C CNN "LCSC"
-	1    6250 4200
-	-1   0    0    1
-$EndComp
-Wire Wire Line
-	6250 4050 6250 3800
-Wire Wire Line
-	6250 4350 6250 4600
-$Comp
 L Q_PNP_EBC Q26
 U 1 1 60D53A6B
@@
 Wire Wire Line
 	5950 4050 5950 3200
+$Comp
+L C_Small C16
+U 1 1 60DC3367
+P 4900 2800
+F 0 "C16" V 5000 2750 50  0000 L CNN
+F 1 "NC" V 4800 2650 50  0000 L CNN
+F 2 "Capacitors_THT:C_Disc_D5.0mm_W2.5mm_P5.00mm" H 4900 2800 50  0001 C CNN
+F 3 "" H 4900 2800 50  0001 C CNN
+F 4 "C366798" V 4900 2800 60  0001 C CNN "LCSC"
+	1    4900 2800
+	1    0    0    -1
+$EndComp
+$Comp
+L GND #PWR019
+U 1 1 610036C8
+P 4650 2650
+F 0 "#PWR019" H 4650 2400 50  0001 C CNN
+F 1 "GND" H 4650 2500 50  0000 C CNN
+F 2 "" H 4650 2650 50  0001 C CNN
+F 3 "" H 4650 2650 50  0001 C CNN
+	1    4650 2650
+	1    0    0    -1
+$EndComp
+Wire Wire Line
+	4650 2650 4650 2600
+Wire Wire Line
+	4650 2600 4900 2600
+Wire Wire Line
+	4900 2600 4900 2700
 $EndSCHEMATC
